File: Hardware/Kicad/L-StarLite/L-Star.sch (KiCad schematic (older format))
At the start: 34 parts, among them IC1 24LC512, IC2 WDC 65C02, IC3 P8X32A, IC4 LM1086-5.0, IC5 LM1086-3.3, P1 PROP PLUG, P2 PS/2 KBD, P3 TV OUT, P4 POWER IN, SW1 RESET, SW2 RESET6502, U1 OSHW Logo, X1 5MHz

Commit message: Updated L-Star Lite
Designed a PCB for L-Star Lite
Also updated KiCad to 5.0.1.4 which insists on creating "rescue" libraries from the old files. I'll figure out how to clean everything up later.
Parts:
- removed C6: 47u, Discret:C1V7, symbol CP1
- removed IC4: LM1086-5.0, 00Jac:00JG-TO-220_Neutral123_Horizontal_LargePads-Heatsink, symbol LM1086
- C1, C2, C3, C4, C5: symbol C -> L-Star-rescue:C-jac
- C6: renamed from C7; footprint Discret:C1V7 -> 00Jac:00JG-C1V7; symbol CP1 -> L-Star-rescue:CP1-jac
- C7: renamed from C8; footprint Discret:C1V7 -> 00Jac:00JG-C1V7; symbol CP1 -> L-Star-rescue:CP1-jac
- D1: symbol LED -> L-Star-rescue:LED-jac
- IC1: footprint Sockets_DIP:DIP-8__300 -> 00Jac:00JG-DIP-8__300; symbol 24LC -> L-Star-rescue:24LC-jac
- IC2: footprint Sockets_DIP:DIP-40__600 -> 00Jac:00JG-DIP-40__600; symbol 65(C)02 -> L-Star-rescue:65(C)02-jac
- IC3: footprint Sockets_DIP:DIP-40__600 -> 00Jac:00JG-DIP-40__600; symbol P8X32A-DIP -> L-Star-rescue:P8X32A-DIP-jac
- IC4: renamed from IC5; footprint 00Jac:00JG-TO-220_Neutral123_Horizontal_LargePads-Heatsink -> 00Jac:00JG-TO-220_Neutral123_Upright_LargePads; symbol LM1086 -> L-Star-rescue:LM1086-jac
- P1: footprint Pin_Headers:Pin_Header_Angled_1x04 -> 00Jac:00JG-Pin_Header_Angled_1x04; symbol CONN_4 -> L-Star-rescue:CONN_4-jac
- P2: symbol CONN_6 -> L-Star-rescue:CONN_6-jac
- P3: symbol CONN_2 -> L-Star-rescue:CONN_2-jac
- P4: value POWER IN -> 5V IN; symbol BARREL_JACK -> L-Star-rescue:BARREL_JACK-L-Star-rescue
- R1, R10, R11, R12, R2, R3, R4, R5, R6, R7, R8, R9: footprint Discret:R3 -> 00Jac:00JG-R300; symbol R -> L-Star-rescue:R-jac
- SW1, SW2: symbol SW_PUSH -> L-Star-rescue:SW_PUSH-jac
- U1: symbol Dummy -> L-Star-rescue:Dummy-jac
- X1: symbol XTAL -> L-Star-rescue:XTAL-jac
Connections:
- net labels added: +5V
- net labels removed: +5C
- wire segments 153 -> 197
Other:
- moved on the sheet: P4
